File: JLink-OB-RA.kicad_pcb (KiCad board)
At the start: 4 copper layers, 35 x 13.5 mm, 49 parts, among them J1 USB_C_Receptacle_USB2.0, J2 Conn_02x05_Counter_Clockwise, J3 DBG, U1 R7FA4M2AB3CNE#AA0, U2 ESD0524P_C2901307, U3 TTP223, U4 TTP223, U5 RS2227XUTQK10, U6 RS2227XUTQK10, U7 ME6211C33M5G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

Commit message: update: 更新为1.1.0
Parts:
- added C15: 10u, Capacitor_SMD:C_0402_1005Metric, F.Cu at (22.1, 26.6)
- added C16: 22u, Capacitor_SMD:C_0603_1608Metric, F.Cu at (19.0, 18.6)
- added C17: 0.1u, Capacitor_SMD:C_0402_1005Metric, F.Cu at (20.2, 19.1)
- added C18: 10u, Capacitor_SMD:C_0402_1005Metric, F.Cu at (24.0, 21.5)
- added L1: 2.2u, Inductor_SMD:L_1008_2520Metric, F.Cu at (25.5, 17.9)
- added R17: 100k, Resistor_SMD:R_0402_1005Metric, F.Cu at (18.8, 16.6)
- added R18: 22.1k, Resistor_SMD:R_0402_1005Metric, F.Cu at (20.2, 17.0)
- added R21: 6.8k, Resistor_SMD:R_0402_1005Metric, F.Cu at (22.1, 21.5)
- added U8: MT9700, Package_TO_SOT_SMD:SOT-23-5, F.Cu at (23.1, 24.1)
- C10: value 1u -> 22p
- C11: value 1u -> 22u; footprint Capacitor_SMD:C_0402_1005Metric -> Capacitor_SMD:C_0603_1608Metric
- D1: footprint LED_SMD:LED_0603_1608Metric -> LED_SMD:LED_0402_1005Metric
- J1: footprint Connector_USB:USB_C_Receptacle_G-Switch_GT-USB-7010ASV -> My USB Connector:USB-C-SMD_SHOU_TYPE-C-16P-CB1.6
- U1: value R7FA4M2AB3CNE#AA0 -> R7FA4M2AB3CFL#AA0; footprint Package_DFN_QFN:QFN-48-1EP_7x7mm_P0.5mm_EP3.5x3.5mm -> Package_QFP:LQFP-48_7x7mm_P0.5mm
- U7: value ME6211C33M5G -> MT3410
- Y1: footprint Crystal:Crystal_SMD_2016-4Pin_2.0x1.6mm -> Crystal:Crystal_SMD_2520-4Pin_2.5x2.0mm
- moved R10 11.6 mm to (17.0, 27.0), turned to -90 degrees
- moved R9 7.29 mm to (22.1, 20.5)
- moved C10 6.94 mm to (17.8, 18.1), turned to -90 degrees
- moved R13 6.59 mm to (24.0, 28.7)
- moved R12 6.54 mm to (25.9, 28.7)
- moved C13 5.97 mm to (18.4, 23.6)
- moved C14 5.97 mm to (18.4, 24.6)
- moved R3 5.95 mm to (20.3, 20.5)
- moved U2 5.95 mm to (18.4, 21.7)
- moved R4 5.95 mm to (20.3, 21.5)
- moved R5 5.95 mm to (20.3, 22.5)
- moved R6 5.94 mm to (20.3, 23.6)
- moved R7 5.93 mm to (20.3, 24.6)
- moved C12 5.93 mm to (18.4, 25.6)
- moved R16 5.93 mm to (20.3, 25.6)
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Connections:
- C10 pad 1: VBUS -> +3V3
- C10 pad 2: GND -> Net-(U7-FB)
- J2 pad 10: /#RESET -> /TDO
- J2 pad 6: /TDO -> /#RESET
- U2 pad 1: /USB_D- -> GND
- U2 pad 10: /USB_D- -> GND
- U2 pad 2: /USB_D+ -> /USB_D-
- U2 pad 4: GND -> /USB_D+
- U2 pad 7: GND -> /USB_D+
- U2 pad 9: /USB_D+ -> /USB_D-
- U7 pad 1: VBUS -> +5V
- U7 pad 3: VBUS -> Net-(U7-SW)
- U7 pad 4: unconnected-(U7-NC-Pad4) -> +5V
- U7 pad 5: +3V3 -> Net-(U7-FB)
Routing:
- net GND: track 17.2 -> 48.7 mm, vias 27 -> 41
- net +5V: track 0.00 -> 15.8 mm, vias 0 -> 2
- net /TRST: track 23.6 -> 32.0 mm, vias 3 -> 1
- net +3V3: track 127.7 -> 135.7 mm, vias 16 -> 17
- net Net-(U1-USB_DP): track 1.26 -> 9.18 mm, vias 0 -> 2
- net Net-(U1-P111): track 19.8 -> 11.9 mm
- net /TCK: track 16.1 -> 24.0 mm
- net /RA_DIO: track 5.41 -> 13.1 mm, vias 0 -> 1
- net Net-(U1-P102): track 2.58 -> 10.0 mm, vias 0 -> 2
- net Net-(U1-USB_DM): track 1.10 -> 8.20 mm, vias 0 -> 2
- net Net-(J1-CC2): track 10.6 -> 3.61 mm, vias 2 -> 0
- net Net-(U1-P101): track 1.58 -> 8.36 mm, vias 0 -> 2
- net /TDO: track 22.5 -> 16.0 mm
- net Net-(U1-P112): track 3.93 -> 9.62 mm, vias 0 -> 2
- net Net-(U3-I): track 5.24 -> 0.00 mm
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Other:
- board size 35 x 13.5 mm -> 40 x 13.5 mm
- board text removed: "V1.0.0"

Commit message: update
Parts:
- J3: value DBG -> Header; footprint Connector_PinHeader_1.27mm:PinHeader_1x04_P1.27mm_Vertical -> Connector_PinHeader_1.00mm:PinHeader_1x02_P1.00mm_Vertical
- moved J3 8.56 mm to (26.4, 30.4)
- moved C18 8.48 mm to (32.3, 23.5)
- moved TP1 8.48 mm to (46.5, 30.5)
- moved U3 8.48 mm to (46.6, 27.8)
- moved U4 8.48 mm to (46.6, 21.0)
- moved C2 8.48 mm to (41.6, 18.7)
- moved C3 8.48 mm to (37.3, 19.0)
- moved C4 8.48 mm to (49.1, 28.6)
- moved C5 8.48 mm to (44.0, 28.6)
- moved C9 8.48 mm to (49.1, 26.7)
- moved D2 8.48 mm to (50.6, 29.3)
- moved D3 8.48 mm to (50.6, 19.8)
- moved J1 8.48 mm to (22.5, 24.5)
- moved J2 8.48 mm to (56.4, 29.6)
- moved R11 8.48 mm to (42.5, 30.7)
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Connections:
- J3 pad 1: +3V3 -> /BOOT
- J3 pad 2: /RA_CLK -> GND
- R6 pad 2: Net-(U1-P201/MD) -> /BOOT
- U1 pad 20: Net-(U1-P201/MD) -> /BOOT
- U1 pad 24: /RA_CLK -> unconnected-(U1-P300/TCK/SWCLK-Pad24)
- U1 pad 25: /RA_DIO -> unconnected-(U1-P108/TMS/SWDIO-Pad25)
Routing:
- net /RA_DIO: track 13.1 -> 0.00 mm, vias 1 -> 0
- net /RA_CLK: track 12.9 -> 0.00 mm, vias 1 -> 0
- net /BOOT: track 0.00 -> 11.9 mm, vias 0 -> 1
- net Net-(U1-P201/MD): track 5.89 -> 0.00 mm
- net +3V3: track 135.7 -> 130.6 mm
- net GND: track 48.7 -> 50.2 mm, vias 41 -> 42
- net Net-(U1-P104): track 8.02 -> 9.15 mm
- net Net-(U1-P101): track 8.36 -> 9.12 mm
- net /XTAL: track 6.13 -> 5.43 mm
- net Net-(U1-P200): track 5.71 -> 5.12 mm
- net /USB_D-: track 5.51 -> 4.93 mm
Other:
- board text added: "V1.1.0"
- board text removed: "C"
- board text removed: "D"
- board text removed: "G"
- board text removed: "JLCJLCJLC"
- board text removed: "V"
