File: JLink-OB-RA.kicad_pcb (KiCad board)
At the start: 4 copper layers, 40 x 13.5 mm, 58 parts, among them J1 USB_C_Receptacle_USB2.0, J2 Conn_02x05_Counter_Clockwise, J3 Header, U1 R7FA4M2AB3CFL#AA0, U2 ESD0524P_C2901307, U3 TTP223, U4 TTP223, U5 RS2227XUTQK10, U6 RS2227XUTQK10, U7 MT3410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

Commit message: update: 更新版本
Other:
- board text added: "V1.1.1"
Changed lines of the file:
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@@
 		(layer "Edge.Cuts")
 	)
-	(gr_text "V1.1.0"
+	(gr_text "V1.1.1"
 		(at 28.0416 31.1912 0)
 		(layer "F.Cu")
@@
 			(justify left bottom)
 		)
-		(render_cache "V1.1.0" 0
+		(render_cache "V1.1.1" 0
 			(polygon
 				(pts
@@
 			(polygon
 				(pts
-					(xy 30.809219 30.285868) (xy 30.84945 30.292651) (xy 30.886476 30.304652) (xy 30.920296 30.32187)
-					(xy 30.95091 30.344305) (xy 30.978319 30.371959) (xy 30.993225 30.391055) (xy 31.015242 30.426672)
-					(xy 31.030169 30.45837) (xy 31.042707 30.492915) (xy 31.052857 30.530308) (xy 31.060619 30.570549)
-					(xy 31.065992 30.613637) (xy 31.068455 30.647823) (xy 31.069574 30.68361) (xy 31.069649 30.695895)
-					(xy 31.068977 30.732206) (xy 31.066962 30.766899) (xy 31.062186 30.810635) (xy 31.055021 30.851491)
-					(xy 31.045468 30.889468) (xy 31.033527 30.924565) (xy 31.019198 30.956782) (xy 30.997927 30.993004)
-					(xy 30.993225 30.999708) (xy 30.96774 31.030196) (xy 30.939049 31.055517) (xy 30.907153 31.07567)
-					(xy 30.87205 31.090656) (xy 30.833743 31.100474) (xy 30.792229 31.105125) (xy 30.774726 31.105539)
-					(xy 30.740233 31.103885) (xy 30.700001 31.097167) (xy 30.662976 31.085282) (xy 30.629156 31.068229)
-					(xy 30.598541 31.046009) (xy 30.571133 31.018621) (xy 30.556226 30.999708) (xy 30.53421 30.964386)
-					(xy 30.519283 30.932889) (xy 30.506745 30.898512) (xy 30.496595 30.861255) (xy 30.488833 30.821119)
-					(xy 30.48346 30.778103) (xy 30.480997 30.74395) (xy 30.479877 30.708179) (xy 30.479803 30.695895)
-					(xy 30.665989 30.695895) (xy 30.666682 30.730701) (xy 30.669343 30.769009) (xy 30.673999 30.803543)
-					(xy 30.681953 30.839061) (xy 30.69437 30.873361) (xy 30.712201 30.903197) (xy 30.739063 30.926402)
-					(xy 30.774726 30.935082) (xy 30.810389 30.926402) (xy 30.837251 30.903197) (xy 30.855082 30.873361)
-					(xy 30.867498 30.839061) (xy 30.875453 30.803543) (xy 30.880109 30.769009) (xy 30.88277 30.730701)
-					(xy 30.883463 30.695895) (xy 30.88277 30.661067) (xy 30.880109 30.622679) (xy 30.875453 30.588005)
-					(xy 30.867498 30.552248) (xy 30.855082 30.517573) (xy 30.837251 30.487242) (xy 30.810389 30.463651)
-					(xy 30.774726 30.454827) (xy 30.739063 30.463651) (xy 30.712201 30.487242) (xy 30.69437 30.517573)
-					(xy 30.681953 30.552248) (xy 30.673999 30.588005) (xy 30.669343 30.622679) (xy 30.666682 30.661067)
-					(xy 30.665989 30.695895) (xy 30.479803 30.695895) (xy 30.480474 30.659574) (xy 30.482489 30.624855)
-					(xy 30.487266 30.581054) (xy 30.494431 30.540101) (xy 30.503983 30.501997) (xy 30.515925 30.466739)
-					(xy 30.530254 30.43433) (xy 30.551524 30.397823) (xy 30.556226 30.391055) (xy 30.581711 30.360271)
-					(xy 30.610402 30.334705) (xy 30.642299 30.314356) (xy 30.677401 30.299225) (xy 30.715709 30.289312)
-					(xy 30.757223 30.284616) (xy 30.774726 30.284199)
+					(xy 30.762416 31.091861) (xy 30.580162 31.091861) (xy 30.580162 30.500818) (xy 30.403721 30.591945)
+					(xy 30.403721 30.402852) (xy 30.608543 30.298047) (xy 30.762416 30.298047)
 				)
 			)

Commit message: fix: 版本号丝印的mask层未修改
Other:
- board text removed: "V1.1.0"
Changed lines of the file:
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@@
 		)
 	)
-	(gr_text "V1.1.0"
+	(gr_text "V1.1.1"
 		(at 28.0416 31.1912 0)
 		(layer "F.Mask")
@@
 			(justify left bottom)
 		)
-		(render_cache "V1.1.0" 0
+		(render_cache "V1.1.1" 0
 			(polygon
 				(pts
@@
 			(polygon
 				(pts
-					(xy 30.809219 30.285868) (xy 30.84945 30.292651) (xy 30.886476 30.304652) (xy 30.920296 30.32187)
-					(xy 30.95091 30.344305) (xy 30.978319 30.371959) (xy 30.993225 30.391055) (xy 31.015242 30.426672)
-					(xy 31.030169 30.45837) (xy 31.042707 30.492915) (xy 31.052857 30.530308) (xy 31.060619 30.570549)
-					(xy 31.065992 30.613637) (xy 31.068455 30.647823) (xy 31.069574 30.68361) (xy 31.069649 30.695895)
-					(xy 31.068977 30.732206) (xy 31.066962 30.766899) (xy 31.062186 30.810635) (xy 31.055021 30.851491)
-					(xy 31.045468 30.889468) (xy 31.033527 30.924565) (xy 31.019198 30.956782) (xy 30.997927 30.993004)
-					(xy 30.993225 30.999708) (xy 30.96774 31.030196) (xy 30.939049 31.055517) (xy 30.907153 31.07567)
-					(xy 30.87205 31.090656) (xy 30.833743 31.100474) (xy 30.792229 31.105125) (xy 30.774726 31.105539)
-					(xy 30.740233 31.103885) (xy 30.700001 31.097167) (xy 30.662976 31.085282) (xy 30.629156 31.068229)
-					(xy 30.598541 31.046009) (xy 30.571133 31.018621) (xy 30.556226 30.999708) (xy 30.53421 30.964386)
-					(xy 30.519283 30.932889) (xy 30.506745 30.898512) (xy 30.496595 30.861255) (xy 30.488833 30.821119)
-					(xy 30.48346 30.778103) (xy 30.480997 30.74395) (xy 30.479877 30.708179) (xy 30.479803 30.695895)
-					(xy 30.665989 30.695895) (xy 30.666682 30.730701) (xy 30.669343 30.769009) (xy 30.673999 30.803543)
-					(xy 30.681953 30.839061) (xy 30.69437 30.873361) (xy 30.712201 30.903197) (xy 30.739063 30.926402)
-					(xy 30.774726 30.935082) (xy 30.810389 30.926402) (xy 30.837251 30.903197) (xy 30.855082 30.873361)
-					(xy 30.867498 30.839061) (xy 30.875453 30.803543) (xy 30.880109 30.769009) (xy 30.88277 30.730701)
-					(xy 30.883463 30.695895) (xy 30.88277 30.661067) (xy 30.880109 30.622679) (xy 30.875453 30.588005)
-					(xy 30.867498 30.552248) (xy 30.855082 30.517573) (xy 30.837251 30.487242) (xy 30.810389 30.463651)
-					(xy 30.774726 30.454827) (xy 30.739063 30.463651) (xy 30.712201 30.487242) (xy 30.69437 30.517573)
-					(xy 30.681953 30.552248) (xy 30.673999 30.588005) (xy 30.669343 30.622679) (xy 30.666682 30.661067)
-					(xy 30.665989 30.695895) (xy 30.479803 30.695895) (xy 30.480474 30.659574) (xy 30.482489 30.624855)
-					(xy 30.487266 30.581054) (xy 30.494431 30.540101) (xy 30.503983 30.501997) (xy 30.515925 30.466739)
-					(xy 30.530254 30.43433) (xy 30.551524 30.397823) (xy 30.556226 30.391055) (xy 30.581711 30.360271)
-					(xy 30.610402 30.334705) (xy 30.642299 30.314356) (xy 30.677401 30.299225) (xy 30.715709 30.289312)
-					(xy 30.757223 30.284616) (xy 30.774726 30.284199)
+					(xy 30.762416 31.091861) (xy 30.580162 31.091861) (xy 30.580162 30.500818) (xy 30.403721 30.591945)
+					(xy 30.403721 30.402852) (xy 30.608543 30.298047) (xy 30.762416 30.298047)
 				)
 			)
