File: JLink-OB-RA.kicad_sch (KiCad schematic)
At the start: 48 parts, among them J1 USB_C_Receptacle_USB2.0, J2 Conn_02x05_Counter_Clockwise, J3 DBG, U1 R7FA4M2AB3CNE#AA0, U2 ESD0524P_C2901307, U3 TTP223, U4 TTP223, U5 RS2227XUTQK10, U6 RS2227XUTQK10, U7 ME6211C33M5G, Y1 12M

Commit message: update: 更新为1.1.0
Parts:
- removed C10, C11: 1u, Capacitor_SMD:C_0402_1005Metric, symbol Device:C
- removed U1: R7FA4M2AB3CNE#AA0, Package_DFN_QFN:QFN-48-1EP_7x7mm_P0.5mm_EP3.5x3.5mm, symbol Renesas MCU:R7FA4M2AB3CNE#AA0
- removed U7: ME6211C33M5G, Package_TO_SOT_SMD:SOT-23-5, symbol LDO:ME6211CxxM5G
- added C12: 22p, Capacitor_SMD:C_0402_1005Metric, symbol Device:C
- added C4, C6: 22u, Capacitor_SMD:C_0603_1608Metric, symbol Device:C
- added C5 (x2): 10u, Capacitor_SMD:C_0402_1005Metric, symbol Device:C
- added C5: 0.1u, Capacitor_SMD:C_0402_1005Metric, symbol Device:C
- added L4: 2.2u, Inductor_SMD:L_1008_2520Metric, symbol Device:L
- added R21: 6.8k, Resistor_SMD:R_0402_1005Metric, symbol Device:R
- added R4: 100k, Resistor_SMD:R_0402_1005Metric, symbol Device:R
- added R5: 22.1k, Resistor_SMD:R_0402_1005Metric, symbol Device:R
- added U1: R7FA4M2AB3CFL#AA0, Package_QFP:LQFP-48_7x7mm_P0.5mm, symbol Renesas MCU:R7FA4M2AB3CFL#AA0
- added U4: MT3410, Package_TO_SOT_SMD:SOT-23-5, symbol DCDC Power Chip:MT3410
- added U8: MT9700, Package_TO_SOT_SMD:SOT-23-5, symbol Load Switch:MT9700
- D1: footprint LED_SMD:LED_0603_1608Metric -> LED_SMD:LED_0402_1005Metric
- J1: footprint Connector_USB:USB_C_Receptacle_G-Switch_GT-USB-7010ASV -> My USB Connector:USB-C-SMD_SHOU_TYPE-C-16P-CB1.6
- Y1: footprint Crystal:Crystal_SMD_2016-4Pin_2.0x1.6mm -> Crystal:Crystal_SMD_2520-4Pin_2.5x2.0mm
Connections:
- net #RESET: now also J2.6 (Pin_6); no longer J2.10 (Pin_10)
- net +3V3: now also C12.1, C6.1, L4.1, R4.1, U1.16 (VCC_USB), U1.2 (VBATT), U1.30 (VCC_2), U1.41 (VREFH), U1.42 (AVCC0), U1.45 (VREFH0), U1.9 (VCC_1)
- net EXTAL: now also U1.8 (P212/EXTAL)
- net GND: now also U2.1, U2.10, C4.2, C5.1, C5.2, C5.2, C6.2, R21.1, R5.2, U1.13 (VSS_USB), U1.31 (VSS_2), U1.43 (AVSS0/VREFL), U1.44 (VREFL0), U1.6 (VSS_1), U4.2 (GND), U8.2 (GND); no longer U2.4, U2.7
- net RA_CLK: now also U1.24 (P300/TCK/SWCLK)
- net RA_DIO: now also U1.25 (P108/TMS/SWDIO)
- net RA_RST: now also U1.19 (RES)
- net RX: now also U1.23 (P301)
- net TDI: now also U1.33 (P103)
- net TDO: now also J2.10 (Pin_10); no longer J2.6 (Pin_6)
- net USB_D+: now also U2.4, U2.7; no longer U2.2, U2.9
- net USB_D-: now also U2.2, U2.9; no longer U2.1, U2.10
- net VBUS: now also C5.1, U8.4 (EN), U8.5 (VIN)
- net XTAL: now also U1.7 (P213/XTAL)
- net at C1.2: now also U1.3 (VCL)
- net at R6.2: now also U1.20 (P201/MD)
- net at R14.1: now also U1.32 (P104)
- net at R8.1: now also U1.28 (P111)
- net at R12.1: now also U1.35 (P101)
- net at R11.1: now also U1.36 (P100)
- net at R7.2: now also U1.21 (P200)
- net at R4.2: now also U1.15 (USB_DP)
- net at R15.1: now also U1.29 (P112)
- net at R2.2: now also U1.12 (P407)
- net at R3.2: now also U1.14 (USB_DM)
- net at R16.2: now also U1.22 (P302)
- net at R13.1: now also U1.34 (P102)
- net at R1.2: now also U1.4 (XCIN)
- new net: L4.2, U4.3 (SW)
- new net: C12.2, R4.2, R5.1, U4.5 (FB)
- new net: R21.2, U8.3 (SET)
- new net +5V: C4.1, C5.1, C5.2, U4.1 (EN), U4.4 (VIN), U8.1 (VOUT)

Commit message: update
Parts:
- removed J3: DBG, Connector_PinHeader_1.27mm:PinHeader_1x04_P1.27mm_Vertical, symbol Connector_Generic:Conn_01x04
- added J3: Header, Connector_PinHeader_1.00mm:PinHeader_1x02_P1.00mm_Vertical, symbol Connector_Generic:Conn_01x02
- added U10: STM32H7A3AGIxQ, Package_BGA:UFBGA-169_7x7mm_Layout13x13_P0.5mm, symbol MCU_ST_STM32H7:STM32H7A3AGIxQ
- added U9: HPM5301IEG1, Package_DFN_QFN:QFN-48-1EP_6x6mm_P0.4mm_EP4.2x4.2mm, symbol HPM5300_Library:HPM5301IEG1
Connections:
- net GND: now also J3.2 (Pin_2)
- net BOOT: now reaches R6.2, U1.20 (P201/MD)
- net BOOT: now also J3.1 (Pin_1)
- net RA_CLK: no longer names the net of U1.24 (P300/TCK/SWCLK)
- net RA_DIO: no longer names the net of U1.25 (P108/TMS/SWDIO)
- new net: U10.B10 (VSS), U10.B3 (VSS), U10.B7 (VSS), U10.C12 (VSS), U10.D2 (VSS), U10.G2 (VSS), U10.H12 (VSS), U10.L12 (VSS), U10.M11 (VSS), U10.M2 (VSS), U10.M4 (VSS), U10.M7 (VSS)
- no-connect marks 17 -> 19
